File: UccMicroDuino/UccMicroDuino.kicad_pcb (KiCad board)
At the start: 2 copper layers, 8 parts, among them J1 Conn_01x10_Socket, J2 USB_A, U1 ATtiny85-20S

Commit message: RUTEO CASI TERMINADO 1 FALTANTE
Parts:
- added D4: LED_GREEN, ledSmd:ledSMD, F.Cu at (110.5, 96.8)
- added D5: D_Zener 3.6V 1/2mW, Diode_SMD:D_SOD-123, F.Cu at (81.0, 76.5)
- added R2: R 330Q 5% 1/8W, Resistor_SMD:R_0805_2012Metric_Pad1.20x1.40mm_HandSolder, F.Cu at (109.0, 78.0)
- added R3: R 330Q 5% 1/8W, Resistor_SMD:R_0805_2012Metric_Pad1.20x1.40mm_HandSolder, F.Cu at (110.0, 89.5)
- added R4: R 68Q 5% 1/8W, Resistor_SMD:R_0805_2012Metric_Pad1.20x1.40mm_HandSolder, F.Cu at (83.5, 76.8)
- added R5: R 68Q 5% 1/8W, Resistor_SMD:R_0805_2012Metric_Pad1.20x1.40mm_HandSolder, F.Cu at (74.5, 76.3)
- C1: value C -> C 0.1u
- D1: value D_Filled -> D_Filled PMLL4148L
- D2: value D_Zener -> D_Zener 3.6V 1/2mW
- D3: value LED -> LED_RED
- J1: value Conn_01x10_Socket -> Conn_01x10_Socket HEADER
- J2: value USB_A -> USB_PCB_A
- R1: value R -> R 1.5KQ 5% 1/8W
- moved R1 68.2 mm to (71.0, 79.2), turned to -90 degrees
- moved D1 60.1 mm to (71.0, 74.0), turned to 90 degrees
- moved J2 57.5 mm to (75.0, 64.2), turned to -90 degrees
- moved D2 53.7 mm to (77.5, 76.5), turned to -90 degrees
- moved U1 41.0 mm to (91.3, 89.4)
- moved C1 39.5 mm to (106.0, 89.5), turned to 180 degrees
- moved J1 37.9 mm to (103.1, 99.5), turned to -90 degrees
- moved D3 27.7 mm to (108.7, 83.4), turned to -90 degrees
Connections:
- C1 pad 1: unconnected-(C1-Pad1) -> +5V
- C1 pad 2: unconnected-(C1-Pad2) -> GND
- D1 pad 2: unconnected-(D1-A-Pad2) -> Net-(D1-A)
- D2 pad 1: unconnected-(D2-K-Pad1) -> Net-(D2-K)
- D2 pad 2: unconnected-(D2-A-Pad2) -> GND
- D3 pad 1: unconnected-(D3-K-Pad1) -> Net-(D3-K)
- D3 pad 2: unconnected-(D3-A-Pad2) -> +5V
- J1 pad 1: unconnected-(J1-Pin_1-Pad1) -> +5V
- J1 pad 2: unconnected-(J1-Pin_2-Pad2) -> GND
- J1 pad 4: unconnected-(J1-Pin_4-Pad4) -> Net-(J1-Pin_4)
- J1 pad 5: unconnected-(J1-Pin_5-Pad5) -> Net-(D4-A)
- J1 pad 6: unconnected-(J1-Pin_6-Pad6) -> Net-(J1-Pin_6)
- J1 pad 7: unconnected-(J1-Pin_7-Pad7) -> Net-(J1-Pin_7)
- J1 pad 8: unconnected-(J1-Pin_8-Pad8) -> Net-(J1-Pin_8)
- J1 pad 9: unconnected-(J1-Pin_9-Pad9) -> Net-(J1-Pin_9)
- J2 pad 1: unconnected-(J2-VBUS-Pad1) -> Net-(D1-A)
- J2 pad 2: unconnected-(J2-D--Pad2) -> Net-(D2-K)
- J2 pad 3: unconnected-(J2-D+-Pad3) -> Net-(D5-K)
- J2 pad 4: unconnected-(J2-GND-Pad4) -> GND
- R1 pad 2: unconnected-(R1-Pad2) -> Net-(D2-K)
- U1 pad 1: unconnected-(U1-~{RESET}/PB5-Pad1) -> Net-(J1-Pin_9)
- U1 pad 2: unconnected-(U1-XTAL1/PB3-Pad2) -> Net-(J1-Pin_7)
- U1 pad 3: unconnected-(U1-XTAL2/PB4-Pad3) -> Net-(J1-Pin_8)
- U1 pad 4: unconnected-(U1-GND-Pad4) -> GND
- U1 pad 5: unconnected-(U1-AREF/PB0-Pad5) -> Net-(J1-Pin_4)
- U1 pad 6: unconnected-(U1-PB1-Pad6) -> Net-(D4-A)
- U1 pad 7: unconnected-(U1-PB2-Pad7) -> Net-(J1-Pin_6)
- U1 pad 8: unconnected-(U1-VCC-Pad8) -> +5V
Routing:
- net GND: track 0.00 -> 118.6 mm
- net Net-(J1-Pin_7): track 0.00 -> 48.7 mm
- net +5V: track 0.00 -> 32.9 mm
- net Net-(D4-A): track 0.00 -> 32.1 mm
- net Net-(J1-Pin_8): track 0.00 -> 30.4 mm
- net Net-(D5-K): track 0.00 -> 28.7 mm
- net Net-(D2-K): track 0.00 -> 21.4 mm
- net Net-(J1-Pin_9): track 0.00 -> 14.7 mm
- net Net-(J1-Pin_6): track 0.00 -> 13.5 mm
- net Net-(D1-A): track 0.00 -> 8.46 mm
- net Net-(J1-Pin_4): track 0.00 -> 8.40 mm
- net Net-(D4-K): track 0.00 -> 5.01 mm
- net Net-(D3-K): track 0.00 -> 2.69 mm
Other:
- board outline added: 45 x 45 mm
