File: UccMicroDuino/UccMicroDuino.kicad_sch (KiCad schematic)
At the start: 8 parts, among them J2 Conn_01x10_Socket, J2 USB_A, U2 ATtiny85-20S

Commit message: RUTEO CASI TERMINADO 1 FALTANTE
Parts:
- added D4: LED_GREEN, ledSmd:ledSMD, symbol Device:LED
- added D5: D_Zener 3.6V 1/2mW, Diode_SMD:D_SOD-123, symbol Device:D_Zener
- added R2, R3: R 330Q 5% 1/8W, Resistor_SMD:R_0805_2012Metric_Pad1.20x1.40mm_HandSolder, symbol Device:R
- added R4, R5: R 68Q 5% 1/8W, Resistor_SMD:R_0805_2012Metric_Pad1.20x1.40mm_HandSolder, symbol Device:R
- C1: value C -> C 0.1u
- D1: value D_Zener -> D_Zener 3.6V 1/2mW
- D3: value LED -> LED_RED
- D5: value D_Filled -> D_Filled PMLL4148L
- J2: value Conn_01x10_Socket -> Conn_01x10_Socket HEADER
- J2: value USB_A -> USB_PCB_A
- R1: value R -> R 1.5KQ 5% 1/8W
Connections:
- net +5V: now also C1.1, D3.2 (A), J2.1 (Pin_1), U2.8 (VCC)
- net GND: now also C1.2, D1.2 (A), J2.2 (Pin_2), J2.4 (GND), U2.4 (GND), D5.2 (A), R2.2, R3.2
- net at D3.1 (K): now also R2.1
- net at R1.2: now also D1.1 (K), J2.2 (D-), R5.2
- net at U2.1 (~{RESET}/PB5): now also J2.9 (Pin_9)
- net at U2.2 (XTAL1/PB3): now also J2.7 (Pin_7), R5.1
- net at U2.3 (XTAL2/PB4): now also J2.8 (Pin_8), R4.1
- net at U2.5 (AREF/PB0): now also J2.4 (Pin_4)
- net at U2.6 (PB1): now also J2.5 (Pin_5), D4.2 (A)
- net at U2.7 (PB2): now also J2.6 (Pin_6)
- net at J2.1 (VBUS): now also D5.2 (A)
- net at J2.3 (D+): now also D5.1 (K), R4.2
- new net: D4.1 (K), R3.1
- no-connect marks 0 -> 2
Other:
- moved on the sheet: D3, U2
