File: proyecto-base-2500352descalzo_zn/UccMicroDuino/UccMicroDuino.kicad_sch (KiCad schematic)
At the start: 14 parts, among them J2 Conn_01x10_Socket HEADER, J2 USB_PCB_A, U2 ATtiny85-20S

Commit message: PLACA EDITADA EN LA ESQUINA
Parts:
- R2, R3: footprint (none) -> Resistor_SMD:R_0805_2012Metric_Pad1.20x1.40mm_HandSolder
Changed lines of the file:
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@@
 			)
 		)
-		(property "Footprint" ""
+		(property "Footprint" "Resistor_SMD:R_0805_2012Metric_Pad1.20x1.40mm_HandSolder"
 			(at 189.23 70.358 90)
 			(effects
@@
 			)
 		)
-		(property "Footprint" ""
+		(property "Footprint" "Resistor_SMD:R_0805_2012Metric_Pad1.20x1.40mm_HandSolder"
 			(at 256.032 88.9 90)
 			(effects

Commit message: Add files via upload
PROYECTO KICAD FINAL TERMINADO.
Other:
- moved on the sheet: D5
Changed lines of the file:
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@@
-	(wire
-		(pts
-			(xy 91.44 110.49) (xy 93.98 110.49)
-		)
-		(stroke
-			(width 0)
-			(type default)
-		)
-	)
 	(wire
 		(pts
@@
 	(wire
 		(pts
-			(xy 85.09 118.11) (xy 91.44 118.11)
+			(xy 85.09 118.11) (xy 93.98 118.11)
 		)
 		(stroke
@@
 	(symbol
 		(lib_id "Device:D_Zener")
-		(at 91.44 114.3 270)
+		(at 93.98 114.3 270)
 		(unit 1)
 		(exclude_from_sim no)
@@
 		(fields_autoplaced yes)
 		(property "Reference" "D5"
-			(at 93.98 113.03 90)
+			(at 96.52 113.03 90)
 			(effects
 				(font
@@
 		)
 		(property "Value" "D_Zener  3.6V 1/2mW"
-			(at 93.98 115.57 90)
+			(at 96.52 115.57 90)
 			(effects
 				(font
@@
 		)
 		(property "Footprint" "Diode_SMD:D_SOD-123"
-			(at 91.44 114.3 0)
+			(at 93.98 114.3 0)
 			(effects
 				(font
@@
 		)
 		(property "Datasheet" "~"
-			(at 91.44 114.3 0)
+			(at 93.98 114.3 0)
 			(effects
 				(font
@@
 		)
 		(property "Description" ""
-			(at 91.44 114.3 0)
-			(effects
-				(font
+			(at 93.98 114.3 0)
+			(effects
+				(font
